File: schematics/pin_interface_circuit/channel_1.kicad_sch (KiCad schematic)
At the start: 9 parts, among them Q10 BSS138, Q11 S9012, Q12 PMBT2222A

Commit message: Signed-off-by: ray33ee <30669752+ray33ee@users.noreply.github.com>
Parts:
- removed R22: 5.6k, Resistor_SMD:R_1206_3216Metric_Pad1.30x1.75mm_HandSolder, symbol Device:R
- added Q13: PMBT2222A, Package_TO_SOT_SMD:SOT-23_Handsoldering, symbol Transistor_BJT:PMBT2222A
- added R25: 2.7k, Resistor_SMD:R_1206_3216Metric_Pad1.30x1.75mm_HandSolder, symbol Device:R
Connections:
- net GND: now also Q13.2 (E)
- net HVS: now also R25.1; no longer R21.2, R23.1
- new net: Q13.3 (C), R21.2, R23.1
- new net: Q13.1 (B), R25.2
Changed lines of the file:
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@@
-	)
-	(junction
-		(at 116.84 87.63)
-		(diameter 0)
-		(color 0 0 0 0)
 	)
 	(junction
@@
 	(wire
 		(pts
-			(xy 115.57 74.93) (xy 115.57 92.71)
+			(xy 115.57 74.93) (xy 115.57 99.06)
 		)
 		(stroke
@@
 	(wire
 		(pts
-			(xy 116.84 100.33) (xy 132.08 100.33)
+			(xy 121.92 100.33) (xy 132.08 100.33)
 		)
 		(stroke
@@
 	(wire
 		(pts
+			(xy 121.92 109.22) (xy 100.33 109.22)
+		)
+		(stroke
+			(width 0)
+			(type default)
+		)
+	)
+	(wire
+		(pts
+			(xy 100.33 99.06) (xy 115.57 99.06)
+		)
+		(stroke
+			(width 0)
+			(type default)
+		)
+	)
+	(wire
+		(pts
 			(xy 95.25 71.12) (xy 102.87 71.12)
 		)
@@
 	(wire
 		(pts
-			(xy 116.84 87.63) (xy 116.84 92.71)
-		)
-		(stroke
-			(width 0)
-			(type default)
-		)
-	)
-	(wire
-		(pts
 			(xy 102.87 71.12) (xy 102.87 73.66)
 		)
@@
 	(wire
 		(pts
-			(xy 88.9 92.71) (xy 115.57 92.71)
-		)
-		(stroke
-			(width 0)
-			(type default)
-		)
-	)
-	(wire
-		(pts
 			(xy 110.49 66.04) (xy 110.49 73.66)
+		)
+		(stroke
+			(width 0)
+			(type default)
+		)
+	)
+	(wire
+		(pts
+			(xy 121.92 100.33) (xy 121.92 109.22)
 		)
 		(stroke
@@
 	(hierarchical_label "HVS"
 		(shape input)
-		(at 88.9 92.71 180)
+		(at 85.09 104.14 180)
 		(fields_autoplaced yes)
 		(effects
@@
 	)
 	(symbol
+		(lib_id "Device:R")
+		(at 88.9 104.14 90)
+		(unit 1)
+		(exclude_from_sim no)
+		(in_bom yes)
+		(on_board yes)
+		(dnp no)
+		(property "Reference" "R25"
+			(at 88.9 101.346 90)
+			(effects
+				(font
+					(size 1.27 1.27)
+				)
+			)
+		)
+		(property "Value" "2.7k"
+			(at 88.9 106.934 90)
+			(effects
+				(font
+					(size 1.27 1.27)
+				)
+			)
+		)
+		(property "Footprint" "Resistor_SMD:R_1206_3216Metric_Pad1.30x1.75mm_HandSolder"
+			(at 88.9 105.918 90)
+			(effects
+				(font
+					(size 1.27 1.27)
+				)
+				(hide yes)
+			)
+		)
+		(property "Datasheet" "~"
+			(at 88.9 104.14 0)
+			(effects
+				(font
+					(size 1.27 1.27)
+				)
+				(hide yes)
+			)
+		)
+		(property "Description" "Resistor"
+			(at 88.9 104.14 0)
+			(effects
+				(font
+					(size 1.27 1.27)
+				)
+				(hide yes)
+			)
+		)
+		(pin "2"
+		)
+		(pin "1"
+		)
+		(instances
+			(project "pin_interface_circuit"
+				(path "/d9377666-f2d1-4dae-8d39-2f1a118a68e8/1d56b778-1640-4c75-8b34-80f290e6101f"
+					(reference "R28")
+					(unit 1)
+				)
+				(path "/d9377666-f2d1-4dae-8d39-2f1a118a68e8/9c35f873-0ee7-4fea-97e8-4782a4e0a1d1"
+					(reference "R25")
+					(unit 1)
+				)
+				(path "/d9377666-f2d1-4dae-8d39-2f1a118a68e8/e1bd20c4-bf72-4d16-a9c6-4b4a98d7de5a"
+					(reference "R27")
+					(unit 1)
+				)
+				(path "/d9377666-f2d1-4dae-8d39-2f1a118a68e8/e7d7fb5b-4b66-4e1d-8b29-c7fe6ba9a236"
+					(reference "R26")
+					(unit 1)
+				)
+			)
+		)
+	)
+	(symbol
 		(lib_id "Device:Q_PNP_BEC")
 		(at 129.54 74.93 0)
@@
 				(path "/d9377666-f2d1-4dae-8d39-2f1a118a68e8/e7d7fb5b-4b66-4e1d-8b29-c7fe6ba9a236"
 					(reference "Q4")
-					(unit 1)
-				)
-			)
-		)
-	)
-	(symbol
-		(lib_id "Device:R")
-		(at 116.84 96.52 0)
-		(unit 1)
-		(exclude_from_sim no)
-		(in_bom yes)
-		(on_board yes)
-		(dnp no)
-		(property "Reference" "R22"
-			(at 113.03 94.742 0)
-			(effects
-				(font
-					(size 1.27 1.27)
-				)
-				(justify left)
-			)
-		)
-		(property "Value" "5.6k"
-			(at 118.364 94.742 0)
-			(effects
-				(font
-					(size 1.27 1.27)
-				)
-				(justify left)
-			)
-		)
-		(property "Footprint" "Resistor_SMD:R_1206_3216Metric_Pad1.30x1.75mm_HandSolder"
-			(at 115.062 96.52 90)
-			(effects
-				(font
-					(size 1.27 1.27)
-				)
-				(hide yes)
-			)
-		)
-		(property "Datasheet" "~"
-			(at 116.84 96.52 0)
-			(effects
-				(font
-					(size 1.27 1.27)
-				)
-				(hide yes)
-			)
-		)
-		(property "Description" "Resistor"
-			(at 116.84 96.52 0)
-			(effects
-				(font
-					(size 1.27 1.27)
-				)
-				(hide yes)
-			)
-		)
-		(pin "2"
-		)
-		(pin "1"
-		)
-		(instances
-			(project "pin_interface_circuit"
-				(path "/d9377666-f2d1-4dae-8d39-2f1a118a68e8/1d56b778-1640-4c75-8b34-80f290e6101f"
-					(reference "R22")
-					(unit 1)
-				)
-				(path "/d9377666-f2d1-4dae-8d39-2f1a118a68e8/9c35f873-0ee7-4fea-97e8-4782a4e0a1d1"
-					(reference "R4")
-					(unit 1)
-				)
-				(path "/d9377666-f2d1-4dae-8d39-2f1a118a68e8/e1bd20c4-bf72-4d16-a9c6-4b4a98d7de5a"
-					(reference "R16")
-					(unit 1)
-				)
-				(path "/d9377666-f2d1-4dae-8d39-2f1a118a68e8/e7d7fb5b-4b66-4e1d-8b29-c7fe6ba9a236"
-					(reference "R10")
 					(unit 1)
 				)
@@
 					(unit 1)
 				)
+			)
+		)
+	)
+	(symbol
+		(lib_id "Transistor_BJT:PMBT2222A")
+		(at 97.79 104.14 0)
+		(unit 1)
+		(exclude_from_sim no)
+		(in_bom yes)
+		(on_board yes)
+		(dnp no)
+		(fields_autoplaced yes)
+		(property "Reference" "Q13"
+			(at 102.87 102.8699 0)
+			(effects
+				(font
+					(size 1.27 1.27)
+				)
+				(justify left)
+			)
+		)
+		(property "Value" "PMBT2222A"
+			(at 102.87 105.4099 0)
+			(effects
+				(font
+					(size 1.27 1.27)
+				)
+				(justify left)
+			)
+		)
+		(property "Footprint" "Package_TO_SOT_SMD:SOT-23_Handsoldering"
+			(at 102.87 106.045 0)
+			(effects
+				(font
+					(size 1.27 1.27)
+					(italic yes)
+				)
+				(justify left)
+				(hide yes)
+			)
+		)
+		(property "Datasheet" "https://assets.nexperia.com/documents/data-sheet/PMBT2222A.pdf"
+			(at 97.79 104.14 0)
+			(effects
+				(font
+					(size 1.27 1.27)
+				)
+				(justify left)
+				(hide yes)
+			)
+		)
+		(property "Description" "600mA Ic, 40V Vce, NPN Transistor, SOT-23"
+			(at 97.79 104.14 0)
+			(effects
+				(font
+					(size 1.27 1.27)
+				)
+				(hide yes)
+			)
+		)
+		(pin "2"
+		)
+		(pin "3"
+		)
+		(pin "1"
+		)
+		(instances
+			(project "pin_interface_circuit"
+				(path "/d9377666-f2d1-4dae-8d39-2f1a118a68e8/1d56b778-1640-4c75-8b34-80f290e6101f"
+					(reference "Q16")
+					(unit 1)
+				)
+				(path "/d9377666-f2d1-4dae-8d39-2f1a118a68e8/9c35f873-0ee7-4fea-97e8-4782a4e0a1d1"
+					(reference "Q13")
+					(unit 1)
+				)
+				(path "/d9377666-f2d1-4dae-8d39-2f1a118a68e8/e1bd20c4-bf72-4d16-a9c6-4b4a98d7de5a"
+					(reference "Q15")
+					(unit 1)
+				)
+				(path "/d9377666-f2d1-4dae-8d39-2f1a118a68e8/e7d7fb5b-4b66-4e1d-8b29-c7fe6ba9a236"
+					(reference "Q14")
+					(unit 1)
+				)
