File: schematics/micro/pic1.kicad_sch (KiCad schematic)
At the start: 10 parts, among them Q11 PMBT2222A, Q12 BSS138, Q13 S9012, Q14 PMBT2222A

Commit message: Signed-off-by: Ray33ee <30669752+ray33ee@users.noreply.github.com>
Parts:
- renumbered Q11 to Q1, Q12 to Q2, Q13 to Q3, Q14 to Q4, R23 to R3, R24 to R4, R25 to R5, R26 to R6, R27 to R7, R28 to R8
Changed lines of the file:
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@@
 (kicad_sch
-	(version 20231120)
+	(version 20250114)
 	(generator "eeschema")
-	(generator_version "8.0")
+	(generator_version "9.0")
 	(paper "A4")
 	(junction
@@
 		(shape input)
 		(at 101.6 100.33 180)
-		(fields_autoplaced yes)
 		(effects
 			(font
@@
 		(shape input)
 		(at 162.56 100.33 0)
-		(fields_autoplaced yes)
 		(effects
 			(font
@@
 		(shape input)
 		(at 97.79 123.19 180)
-		(fields_autoplaced yes)
 		(effects
 			(font
@@
 		(shape input)
 		(at 101.6 106.68 180)
-		(fields_autoplaced yes)
 		(effects
 			(font
@@
 		(on_board yes)
 		(dnp no)
-		(property "Reference" "R25"
+		(property "Reference" "R5"
 			(at 124.714 98.298 0)
 			(effects
@@
 		(on_board yes)
 		(dnp no)
-		(property "Reference" "R27"
+		(property "Reference" "R7"
 			(at 133.35 91.186 90)
 			(effects
@@
 		(dnp no)
 		(fields_autoplaced yes)
-		(property "Reference" "Q14"
+		(property "Reference" "Q4"
 			(at 147.32 105.4099 0)
 			(effects
@@
 		(on_board yes)
 		(dnp no)
-		(property "Reference" "R23"
+		(property "Reference" "R3"
 			(at 101.6 120.396 90)
 			(effects
@@
 		(on_board yes)
 		(dnp no)
-		(property "Reference" "R24"
+		(property "Reference" "R4"
 			(at 109.474 93.726 0)
 			(effects
@@
 		(on_board yes)
 		(dnp no)
-		(property "Reference" "R28"
+		(property "Reference" "R8"
 			(at 133.35 103.886 90)
 			(effects
@@
 		(dnp no)
 		(fields_autoplaced yes)
-		(property "Reference" "#PWR016"
+		(property "Reference" "#PWR010"
 			(at 144.78 128.27 0)
 			(effects
@@
 		(on_board yes)
 		(dnp no)
-		(property "Reference" "Q12"
+		(property "Reference" "Q2"
 			(at 119.126 96.774 90)
 			(effects
@@
 		(on_board yes)
 		(dnp no)
-		(property "Reference" "Q13"
+		(property "Reference" "Q3"
 			(at 147.32 95.2501 0)
 			(effects
@@
 		(dnp no)
 		(fields_autoplaced yes)
-		(property "Reference" "Q11"
+		(property "Reference" "Q1"
 			(at 115.57 121.9199 0)
 			(effects
@@
 		(on_board yes)
 		(dnp no)
-		(property "Reference" "R26"
+		(property "Reference" "R6"
 			(at 124.46 87.122 0)
 			(effects
