File: schematics/micro/micro.kicad_sch (KiCad schematic)
At the start: 22 parts, among them J1 16-pin ZIF Socket, Q5 PMBT2222A, Q6 CJ2301, U1 NUCLEO-G474RE, U2 MCP23017_SO, U3 MCP23017_SO

Commit message: Signed-off-by: ray33ee <30669752+ray33ee@users.noreply.github.com>
Parts:
- added Q67: CJ2301, Package_TO_SOT_SMD:SOT-23, symbol Transistor_FET:IRF4905
- added Q68: PMBT2222A, Package_TO_SOT_SMD:SOT-23, symbol Transistor_BJT:PMBT2222A
- added R107, R108: R, Resistor_SMD:R_1206_3216Metric_Pad1.30x1.75mm_HandSolder, symbol Device:R
- added R109: 2k2, Resistor_SMD:R_1206_3216Metric_Pad1.30x1.75mm_HandSolder, symbol Device:R
Connections:
- new net: Q67.2 (S), R107.2
- new net: Q67.1 (G), Q68.3 (C)
- new net: Q67.3 (D), R108.1
- new net: Q68.1 (B), R109.1
- no-connect marks 43 -> 47

Commit message: Signed-off-by: Ray33ee <30669752+ray33ee@users.noreply.github.com>
Changed lines of the file:
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@@
 	(wire
 		(pts
-			(xy 105.41 46.99) (xy 92.71 46.99)
-		)
-		(stroke
-			(width 0)
-			(type default)
-		)
-	)
-	(wire
-		(pts
 			(xy 48.26 40.64) (xy 41.91 40.64)
 		)
@@
 	(wire
 		(pts
+			(xy 82.55 46.99) (xy 105.41 46.99)
+		)
+		(stroke
+			(width 0)
+			(type default)
+		)
+	)
+	(wire
+		(pts
 			(xy 179.07 53.34) (xy 179.07 68.58)
 		)
@@
 	(symbol
 		(lib_id "power:GND")
-		(at 92.71 46.99 0)
+		(at 82.55 46.99 0)
 		(mirror y)
 		(unit 1)
@@
 		(fields_autoplaced yes)
 		(property "Reference" "#PWR07"
-			(at 92.71 53.34 0)
+			(at 82.55 53.34 0)
 			(effects
 				(font
@@
 		)
 		(property "Value" "GND"
-			(at 92.71 52.07 0)
+			(at 82.55 52.07 0)
 			(effects
 				(font
@@
 		)
 		(property "Footprint" ""
-			(at 92.71 46.99 0)
+			(at 82.55 46.99 0)
 			(effects
 				(font
@@
 		)
 		(property "Datasheet" ""
-			(at 92.71 46.99 0)
+			(at 82.55 46.99 0)
 			(effects
 				(font
@@
 		)
 		(property "Description" "Power symbol creates a global label with name \"GND\" , ground"
-			(at 92.71 46.99 0)
+			(at 82.55 46.99 0)
 			(effects
 				(font
