File: schematics/micro/micro.kicad_pcb (KiCad board)
At the start: 2 copper layers, 70 x 120.3 mm, 182 parts, among them J1 16-pin ZIF Socket, Q1 PMBT2222A, Q10 PMBT2222A, Q11 PMBT2222A, Q12 BSS138, Q13 S9012, Q14 PMBT2222A, Q15 PMBT2222A, Q16 BSS138, Q17 S9012, Q18 PMBT2222A, Q19 PMBT2222A, Q2 BSS138, Q20 BSS138, Q21 S9012, Q22 PMBT2222A, Q23 PMBT2222A, Q24 BSS138, Q25 S9012, Q26 PMBT2222A, Q27 PMBT2222A, Q28 BSS138, Q29 S9012, Q3 S9012, Q30 PMBT2222A, Q31 PMBT2222A, Q32 BSS138, Q33 S9012, Q34 PMBT2222A, Q35 PMBT2222A, Q36 BSS138, Q37 S9012, Q38 PMBT2222A, Q39 PMBT2222A, Q4 PMBT2222A, Q40 BSS138, Q41 S9012, Q42 PMBT2222A, Q43 PMBT2222A, Q44 BSS138, Q45 S9012, Q46 PMBT2222A, Q47 PMBT2222A, Q48 BSS138, Q49 S9012, Q5 PMBT2222A, Q50 PMBT2222A, Q51 PMBT2222A, Q52 BSS138, Q53 S9012, Q54 PMBT2222A, Q55 PMBT2222A, Q56 BSS138, Q57 S9012, Q58 PMBT2222A, Q59 PMBT2222A, Q6 CJ2301, Q60 BSS138, Q61 S9012, Q62 PMBT2222A, Q63 PMBT2222A, Q64 BSS138, Q65 S9012, Q66 PMBT2222A, Q7 PMBT2222A, Q8 BSS138, Q9 S9012, U1 NUCLEO-G474RE, U2 MCP23017_SO, U3 MCP23017_SO

Commit message: Signed-off-by: ray33ee <30669752+ray33ee@users.noreply.github.com>
Parts:
- added Q67: CJ2301, Package_TO_SOT_SMD:SOT-23, F.Cu at (178.5, 47.5)
- added Q68: PMBT2222A, Package_TO_SOT_SMD:SOT-23, F.Cu at (174.6, 46.5)
- added R107: R, Resistor_SMD:R_1206_3216Metric_Pad1.30x1.75mm_HandSolder, F.Cu at (174.1, 49.4)
- added R108: R, Resistor_SMD:R_1206_3216Metric_Pad1.30x1.75mm_HandSolder, F.Cu at (179.0, 44.6)
- added R109: 2k2, Resistor_SMD:R_1206_3216Metric_Pad1.30x1.75mm_HandSolder, F.Cu at (170.2, 45.6)
Routing:
- net HV: track 704.1 -> 705.3 mm

Commit message: Signed-off-by: Ray33ee <30669752+ray33ee@users.noreply.github.com>
Other:
- board text added: "- Add vias to island on pin 2 of Q10 - Add Test point for HV - Remove Test circuit (top right)"

Commit message: Signed-off-by: Ray33ee <30669752+ray33ee@users.noreply.github.com>
Other:
- board text added: "- Add vias to island on pin 2 of Q10 - Add Test point for HV - Remove Test circuit (top right) - Write on the front and back of the boards the CN7 and CN10 header names"
- board text removed: "- Add vias to island on pin 2 of Q10 - Add Test point for HV - Remove Test circuit (top right)"
Changed lines of the file:
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@@
 		)
 	)
-	(gr_text "- Add vias to island on pin 2 of Q10\n- Add Test point for HV\n- Remove Test circuit (top right)"
+	(gr_text "- Add vias to island on pin 2 of Q10\n- Add Test point for HV\n- Remove Test circuit (top right)\n- Write on the front and back of the boards the CN7 and CN10 header names"
 		(at 191.000113 53 0)
 		(layer "Eco1.User")
