File: schematics/debug_board/debug/debug.kicad_pcb (KiCad board)
At the start: 2 copper layers, 136.2 x 55.5 mm, 26 parts, among them CN10 Conn_02x19_Odd_Even, CN7 Conn_02x19_Odd_Even, J1 Conn_01x02_Pin, J2 Conn_01x02_Pin, SW2 SW_MISC, U1 NUCLEO-G474RE

Commit message: Signed-off-by: Ray33ee <30669752+ray33ee@users.noreply.github.com>
Parts:
- removed TP1: TestPoint, TestPoint:TestPoint_Pad_2.0x2.0mm
- added J3: Conn_01x04_Pin, Connector_PinHeader_2.54mm:PinHeader_1x04_P2.54mm_Vertical, F.Cu at (58.4, 88.9)
- added JP7: SolderJumper_2_Bridged, Jumper:SolderJumper-2_P1.3mm_Bridged_RoundedPad1.0x1.5mm, B.Cu at (171.9, 120.5)
- D6: renamed from PWM1; value PWM_LED -> LED
- moved D5 4.00 mm to (186.2, 105.2)
- moved D6 4.00 mm to (186.1, 109.2)
- moved JP5 4.00 mm to (183.9, 106.2)
- moved JP6 4.00 mm to (183.9, 110.2)
- moved R5 4.00 mm to (188.1, 106.2)
- moved R6 4.00 mm to (188.1, 110.2)
- moved J1 2.54 mm to (182.9, 81.3), turned to -90 degrees
- moved J2 2.54 mm to (58.4, 116.8), turned to -90 degrees
- renumbered D6 to D5, JP6 to JP5, JP5 to JP6, D4 to PWM1, R6 to R5, R5 to R6
Connections:
- JP5 pad 2: /CN10_16 -> /CN10_12
- JP6 pad 2: /CN10_12 -> /CN10_16
Routing:
- net /CN10_34: track 18.7 -> 22.9 mm
Other:
- board size 136.2 x 55.5 mm -> 139.2 x 55.5 mm
- board text added: "D2"
- board text added: "D3"
- board text added: "D5"
- board text added: "D6"
- board text added: "J1"
- board text added: "J2"
