File: schematics/debug_board/debug/debug.kicad_sch (KiCad schematic)
At the start: 26 parts, among them CN10 Conn_02x19_Odd_Even, CN7 Conn_02x19_Odd_Even, J1 Conn_01x02_Pin, J2 Conn_01x02_Pin, SW2 SW_MISC, U1 NUCLEO-G474RE

Commit message: Signed-off-by: Ray33ee <30669752+ray33ee@users.noreply.github.com>
Parts:
- removed TP1: TestPoint, TestPoint:TestPoint_Pad_2.0x2.0mm, symbol Connector:TestPoint
- added J3: Conn_01x04_Pin, Connector_PinHeader_2.54mm:PinHeader_1x04_P2.54mm_Vertical, symbol Connector:Conn_01x04_Pin
- added JP7: SolderJumper_2_Bridged, Jumper:SolderJumper-2_P1.3mm_Bridged_RoundedPad1.0x1.5mm, symbol Jumper:SolderJumper_2_Bridged
- D6: renamed from PWM1; value PWM_LED -> LED
- renumbered D6 to D5, JP6 to JP5, JP5 to JP6, D4 to PWM1, R6 to R5, R5 to R6
Connections:
- net CN10_12: now also JP5.2 (B); no longer JP6.2 (B)
- net CN10_16: now also JP6.2 (B); no longer JP5.2 (B)
- net CN10_34: now also JP7.1 (A)
- net at SW2.1: now also JP7.2 (B)
- no-connect marks 0 -> 4
Changed lines of the file:
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@@
 		(color 0 0 0 0)
 	)
+	(no_connect
+		(at 227.33 81.28)
+	)
+	(no_connect
+		(at 227.33 88.9)
+	)
+	(no_connect
+		(at 227.33 86.36)
+	)
+	(no_connect
+		(at 227.33 83.82)
+	)
 	(wire
 		(pts
@@
 	(wire
 		(pts
-			(xy 102.87 175.26) (xy 113.03 175.26)
-		)
-		(stroke
-			(width 0)
-			(type default)
-		)
-	)
-	(wire
-		(pts
 			(xy 102.87 50.8) (xy 87.63 50.8)
 		)
@@
 	(wire
 		(pts
+			(xy 105.41 175.26) (xy 113.03 175.26)
+		)
+		(stroke
+			(width 0)
+			(type default)
+		)
+	)
+	(wire
+		(pts
 			(xy 59.69 55.88) (xy 74.93 55.88)
 		)
@@
 	(wire
 		(pts
+			(xy 85.09 175.26) (xy 97.79 175.26)
+		)
+		(stroke
+			(width 0)
+			(type default)
+		)
+	)
+	(wire
+		(pts
 			(xy 59.69 76.2) (xy 74.93 76.2)
 		)
@@
 		)
 	)
-	(label "CN10_16"
+	(label "CN10_12"
 		(at 271.78 138.43 180)
 		(effects
@@
 		)
 	)
+	(label "CN10_34"
+		(at 85.09 175.26 0)
+		(effects
+			(font
+				(size 1.27 1.27)
+			)
+			(justify left bottom)
+		)
+	)
 	(label "CN7_2"
 		(at 102.87 40.64 180)
@@
 		)
 	)
-	(label "CN10_12"
+	(label "CN10_16"
 		(at 271.78 153.67 180)
 		(effects
@@
 		(on_board yes)
 		(dnp no)
-		(property "Reference" "PWM1"
+		(property "Reference" "D6"
 			(at 235.712 150.876 0)
 			(effects
@@
 			)
 		)
-		(property "Value" "PWM_LED"
+		(property "Value" "LED"
 			(at 241.554 150.876 0)
 			(effects
@@
 			(project "debug"
 				(path "/2bcc3c92-74c2-4ef9-b92b-7b4e865bbb22"
-					(reference "PWM1")
+					(reference "D6")
 					(unit 1)
 				)
@@
 		(on_board yes)
 		(dnp no)
-		(property "Reference" "D4"
+		(property "Reference" "PWM1"
 			(at 235.712 128.016 0)
 			(effects
@@
 			(project "debug"
 				(path "/2bcc3c92-74c2-4ef9-b92b-7b4e865bbb22"
-					(reference "D4")
+					(reference "PWM1")
+					(unit 1)
+				)
+			)
+		)
+	)
+	(symbol
+		(lib_id "Jumper:SolderJumper_2_Bridged")
+		(at 101.6 175.26 0)
+		(unit 1)
+		(exclude_from_sim no)
+		(in_bom yes)
+		(on_board yes)
+		(dnp no)
+		(fields_autoplaced yes)
+		(property "Reference" "JP7"
+			(at 101.6 168.91 0)
+			(effects
+				(font
+					(size 1.27 1.27)
+				)
+			)
+		)
+		(property "Value" "SolderJumper_2_Bridged"
+			(at 101.6 171.45 0)
+			(effects
+				(font
+					(size 1.27 1.27)
+				)
+			)
+		)
+		(property "Footprint" "Jumper:SolderJumper-2_P1.3mm_Bridged_RoundedPad1.0x1.5mm"
+			(at 101.6 175.26 0)
+			(effects
+				(font
+					(size 1.27 1.27)
+				)
+				(hide yes)
+			)
+		)
+		(property "Datasheet" "~"
+			(at 101.6 175.26 0)
+			(effects
+				(font
+					(size 1.27 1.27)
+				)
+				(hide yes)
+			)
+		)
+		(property "Description" "Solder Jumper, 2-pole, closed/bridged"
+			(at 101.6 175.26 0)
+			(effects
+				(font
+					(size 1.27 1.27)
+				)
+				(hide yes)
+			)
+		)
+		(pin "1"
+		)
+		(pin "2"
+		)
+		(instances
+			(project ""
+				(path "/2bcc3c92-74c2-4ef9-b92b-7b4e865bbb22"
+					(reference "JP7")
+					(unit 1)
+				)
+			)
+		)
+	)
+	(symbol
+		(lib_id "Connector:Conn_01x04_Pin")
+		(at 222.25 83.82 0)
+		(unit 1)
+		(exclude_from_sim no)
+		(in_bom yes)
+		(on_board yes)
+		(dnp no)
+		(fields_autoplaced yes)
+		(property "Reference" "J3"
+			(at 222.885 76.2 0)
+			(effects
+				(font
+					(size 1.27 1.27)
+				)
+			)
+		)
+		(property "Value" "Conn_01x04_Pin"
+			(at 222.885 78.74 0)
+			(effects
+				(font
+					(size 1.27 1.27)
+				)
+			)
+		)
+		(property "Footprint" "Connector_PinHeader_2.54mm:PinHeader_1x04_P2.54mm_Vertical"
+			(at 222.25 83.82 0)
+			(effects
+				(font
+					(size 1.27 1.27)
+				)
+				(hide yes)
+			)
+		)
+		(property "Datasheet" "~"
+			(at 222.25 83.82 0)
+			(effects
+				(font
+					(size 1.27 1.27)
+				)
+				(hide yes)
+			)
+		)
+		(property "Description" "Generic connector, single row, 01x04, script generated"
+			(at 222.25 83.82 0)
+			(effects
+				(font
+					(size 1.27 1.27)
+				)
+				(hide yes)
+			)
+		)
+		(pin "3"
+		)
+		(pin "1"
+		)
+		(pin "2"
+		)
+		(pin "4"
+		)
+		(instances
+			(project ""
+				(path "/2bcc3c92-74c2-4ef9-b92b-7b4e865bbb22"
+					(reference "J3")
 					(unit 1)
 				)
@@
 		(on_board yes)
 		(dnp no)
-		(property "Reference" "R6"
+		(property "Reference" "R5"
 			(at 245.364 136.398 90)
 			(effects
@@
 			(project "debug"
 				(path "/2bcc3c92-74c2-4ef9-b92b-7b4e865bbb22"
-					(reference "R6")
+					(reference "R5")
 					(unit 1)
 				)
@@
 		(on_board yes)
 		(dnp no)
-		(property "Reference" "R5"
+		(property "Reference" "R6"
 			(at 245.364 151.638 90)
 			(effects
@@
 			(project "debug"
 				(path "/2bcc3c92-74c2-4ef9-b92b-7b4e865bbb22"
-					(reference "R5")
+					(reference "R6")
 					(unit 1)
 				)
@@
 		(on_board yes)
 		(dnp no)
-		(property "Reference" "D6"
+		(property "Reference" "D5"
 			(at 235.712 135.636 0)
 			(effects
@@
 			(project "debug"
 				(path "/2bcc3c92-74c2-4ef9-b92b-7b4e865bbb22"
-					(reference "D6")
+					(reference "D5")
 					(unit 1)
 				)
@@
 		(on_board yes)
 		(dnp no)
-		(property "Reference" "JP6"
+		(property "Reference" "JP5"
 			(at 251.968 133.35 0)
 			(effects
@@
 			(project "debug"
 				(path "/2bcc3c92-74c2-4ef9-b92b-7b4e865bbb22"
-					(reference "JP6")
+					(reference "JP5")
 					(unit 1)
 				)
@@
 		(on_board yes)
 		(dnp no)
-		(property "Reference" "JP5"
+		(property "Reference" "JP6"
 			(at 251.968 148.59 0)
 			(effects
@@
 			(project "debug"
 				(path "/2bcc3c92-74c2-4ef9-b92b-7b4e865bbb22"
-					(reference "JP5")
+					(reference "JP6")
 					(unit 1)
 				)
@@
 					(unit 1)
 				)
-			)
-		)
-	)
-	(symbol
-		(lib_id "Connector:TestPoint")
-		(at 102.87 175.26 0)
-		(unit 1)
-		(exclude_from_sim no)
-		(in_bom yes)
-		(on_board yes)
-		(dnp no)
-		(property "Reference" "TP1"
-			(at 98.552 170.18 0)
-			(effects
-				(font
-					(size 1.27 1.27)
-				)
-				(justify left)
-			)
-		)
-		(property "Value" "TestPoint"
-			(at 103.378 170.18 0)
-			(effects
-				(font
-					(size 1.27 1.27)
-				)
-				(justify left)
-			)
-		)
-		(property "Footprint" "TestPoint:TestPoint_Pad_2.0x2.0mm"
-			(at 107.95 175.26 0)
-			(effects
-				(font
-					(size 1.27 1.27)
-				)
-				(hide yes)
-			)
-		)
-		(property "Datasheet" "~"
-			(at 107.95 175.26 0)
-			(effects
-				(font
-					(size 1.27 1.27)
-				)
-				(hide yes)
-			)
-		)
-		(property "Description" "test point"
-			(at 102.87 175.26 0)
-			(effects
-				(font
-					(size 1.27 1.27)
-				)
-				(hide yes)
-			)
-		)
-		(pin "1"
-		)
-		(instances
-			(project "debug"
-				(path "/2bcc3c92-74c2-4ef9-b92b-7b4e865bbb22"
-					(reference "TP1")
-					(unit 1)
-				)
